Commit message: updated static slam

File: ros2_ws/install/Forklift_Firmware/share/Forklift_Firmware/urdf/my_robot.urdf.xacro (robot description, xacro)
@@ -7,4 +7,7 @@
   <xacro:property name="wheel_radius" value="0.05" />
   <xacro:property name="wheel_width" value="0.04" />
+  <!-- Base Footprint Link -->
+  <link name="base_footprint">
+  </link>
   <!-- Base Link (main body of the robot) -->
   <link name="base_link">
@@ -27,4 +30,10 @@
     </inertial>
   </link>
+  <!-- Joint connecting base_footprint to base_link -->
+  <joint name="base_footprint_joint" type="fixed">
+    <parent link="base_footprint" />
+    <child link="base_link" />
+    <origin xyz="0 0 ${base_height/2}" rpy="0 0 0" />
+  </joint>
   <!-- LiDAR Link -->
   <link name="laser_link">
